File: schematics and PCBs/Main_Schematic_and_PCB/pre_autoRoute.sch (EAGLE design)
At the start: 33 parts, among them IC1 LM386N-1, IC2 LM358N

Commit message: updated main pcb
Parts:
- removed F1: (no value), special:FUSE
Connections:
- removed net N$2: F1.1, JP5.2
- new net N$11: LED3.DO, LED4.DI
- net +12V: now also IC2P.V+, JP5.2; no longer F1.2
- net GND: now also IC2P.V-
Other:
- moved on the sheet: R4
