File: schematics and PCBs/userInterface/clockBot_userInterface.brd (EAGLE design)
At the start: 119.6 x 14.6 mm, 8 parts

Commit message: User interface single row molex
Parts:
- moved JP1 10.5 mm to (63.5, 8.04)
Routing:
- net N$7: track 24.3 -> 32.1 mm
- net N$8: track 46.6 -> 49.7 mm
- net N$1: track 48.0 -> 45.5 mm
- net N$10: track 55.2 -> 52.9 mm
- net N$2: track 29.1 -> 31.4 mm
- net N$6: track 59.1 -> 57.0 mm
- net N$3: track 28.6 -> 27.5 mm
