File: schematics and PCBs/userInterface/clockBot_userInterface.sch (EAGLE design)
At the start: 8 parts

Commit message: finalized PCBs and exported gerbers
Parts:
- R1, R2: device adafruit:FLIPFLOP-RES -> rcl:R-US_0204/7
Connections:
- net N$5 renamed GND
- removed net N$4: FILTER_CUTOFF.S, JP1.7, OCTAVE_SELECT.A
- removed net VDD: R1.1
- new net 5V: FILTER_CUTOFF.S, JP1.7, OCTAVE_SELECT.A, R1.1
Changed lines of the file:
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@@
 <?xml version="1.0" encoding="utf-8"?>
 <!DOCTYPE eagle SYSTEM "eagle.dtd">
-<eagle version="9.5.1">
+<eagle version="9.6.2">
 <drawing>
 <settings>
@@
 <part name="FILTER_CUTOFF" library="pot" library_urn="urn:adsk.eagle:library:331" deviceset="TRIM_US-" device="S64W" package3d_urn="urn:adsk.eagle:package:22708/1" value="1k Ohms"/>
 <part name="OCTAVE_SELECT" library="pot" library_urn="urn:adsk.eagle:library:331" deviceset="TRIM_US-" device="S64W" package3d_urn="urn:adsk.eagle:package:22708/1" value="10K Ohms"/>
-<part name="SUPPLY1" library="supply2" library_urn="urn:adsk.eagle:library:372" deviceset="VDD" device=""/>
 <part name="X_1" library="ngspice-simulation" library_urn="urn:adsk.eagle:library:527439" deviceset="GND" device=""/>
-<part name="R1" library="adafruit" library_urn="urn:adsk.eagle:library:420" deviceset="FLIPFLOP-RES" device="" package3d_urn="urn:adsk.eagle:package:6240726/1" value="100K Ohms"/>
+<part name="R1" library="rcl" library_urn="urn:adsk.eagle:library:334" deviceset="R-US_" device="0204/7" package3d_urn="urn:adsk.eagle:package:23498/2" value="100K Ohms"/>
 <part name="S1" library="switch-omron" library_urn="urn:adsk.eagle:library:377" deviceset="10-XX" device="" package3d_urn="urn:adsk.eagle:package:27496/1"/>
 <part name="C1" library="adafruit" library_urn="urn:adsk.eagle:library:420" deviceset="C-US" device="025-025X050" package3d_urn="urn:adsk.eagle:package:6240323/1" value="50 nF"/>
-<part name="R2" library="adafruit" library_urn="urn:adsk.eagle:library:420" deviceset="FLIPFLOP-RES" device="" package3d_urn="urn:adsk.eagle:package:6240726/1" value="10K Ohms"/>
+<part name="R2" library="rcl" library_urn="urn:adsk.eagle:library:334" deviceset="R-US_" device="0204/7" package3d_urn="urn:adsk.eagle:package:23498/2" value="10K Ohms"/>
 <part name="JP1" library="pinhead" library_urn="urn:adsk.eagle:library:325" deviceset="PINHD-1X8" device="" package3d_urn="urn:adsk.eagle:package:22409/2"/>
 </parts>
@@
 <attribute name="VALUE" x="60.96" y="63.5" size="1.778" layer="96"/>
 </instance>
-<instance part="SUPPLY1" gate="G$1" x="-12.7" y="50.8" smashed="yes">
-<attribute name="VALUE" x="-14.605" y="56.515" size="1.778" layer="96"/>
-</instance>
 <instance part="X_1" gate="G$1" x="-12.7" y="10.16" smashed="yes"/>
 <instance part="R1" gate="G$1" x="-12.7" y="40.64" smashed="yes" rot="R270">
@@
 <wire x1="30.48" y1="33.02" x2="76.2" y2="33.02" width="0.1524" layer="91"/>
 <pinref part="JP1" gate="A" pin="4"/>
+<label x="63.5" y="33.02" size="1.778" layer="95"/>
 </segment>
 </net>
@@
 <wire x1="63.5" y1="55.88" x2="63.5" y2="40.64" width="0.1524" layer="91"/>
 <pinref part="JP1" gate="A" pin="1"/>
+<label x="68.58" y="40.64" size="1.778" layer="95"/>
 </segment>
 </net>
@@
 <wire x1="45.72" y1="35.56" x2="76.2" y2="35.56" width="0.1524" layer="91"/>
 <pinref part="JP1" gate="A" pin="3"/>
+<label x="60.96" y="35.56" size="1.778" layer="95"/>
 </segment>
 </net>
@@
 <wire x1="76.2" y1="30.48" x2="15.24" y2="30.48" width="0.1524" layer="91"/>
 <pinref part="JP1" gate="A" pin="5"/>
-</segment>
-</net>
-<net name="N$4" class="0">
-<segment>
-<pinref part="OCTAVE_SELECT" gate="G$1" pin="A"/>
-<wire x1="22.86" y1="48.26" x2="55.88" y2="48.26" width="0.1524" layer="91"/>
-<wire x1="55.88" y1="48.26" x2="55.88" y2="60.96" width="0.1524" layer="91"/>
-<pinref part="FILTER_CUTOFF" gate="G$1" pin="S"/>
-<wire x1="22.86" y1="48.26" x2="22.86" y2="55.88" width="0.1524" layer="91"/>
-<wire x1="22.86" y1="48.26" x2="22.86" y2="25.4" width="0.1524" layer="91"/>
-<junction x="22.86" y="48.26"/>
-<wire x1="76.2" y1="25.4" x2="22.86" y2="25.4" width="0.1524" layer="91"/>
-<pinref part="JP1" gate="A" pin="7"/>
-</segment>
-</net>
-<net name="N$5" class="0">
+<label x="66.04" y="30.48" size="1.778" layer="95"/>
+</segment>
+</net>
+<net name="GND" class="0">
 <segment>
 <pinref part="VOLUME" gate="G$1" pin="E"/>
@@
 <wire x1="53.34" y1="22.86" x2="76.2" y2="22.86" width="0.1524" layer="91"/>
 <pinref part="JP1" gate="A" pin="8"/>
-</segment>
-</net>
-<net name="VDD" class="0">
-<segment>
-<pinref part="R1" gate="G$1" pin="1"/>
-<pinref part="SUPPLY1" gate="G$1" pin="VDD"/>
-<wire x1="-12.7" y1="48.26" x2="-12.7" y2="45.72" width="0.1524" layer="91"/>
+<label x="66.04" y="22.86" size="1.778" layer="95"/>
 </segment>
 </net>
@@
 <wire x1="38.1" y1="38.1" x2="76.2" y2="38.1" width="0.1524" layer="91"/>
 <pinref part="JP1" gate="A" pin="2"/>
+<label x="68.58" y="38.1" size="1.778" layer="95"/>
 </segment>
 </net>
@@
 <junction x="2.54" y="27.94"/>
 <pinref part="JP1" gate="A" pin="6"/>
+<label x="66.04" y="27.94" size="1.778" layer="95"/>
 </segment>
 </net>
@@
 <wire x1="-10.16" y1="27.94" x2="-12.7" y2="27.94" width="0.1524" layer="91"/>
 <junction x="-12.7" y="27.94"/>
+</segment>
+</net>
+<net name="5V" class="0">
+<segment>
+<pinref part="R1" gate="G$1" pin="1"/>
+<wire x1="-12.7" y1="48.26" x2="-12.7" y2="45.72" width="0.1524" layer="91"/>
+<wire x1="-12.7" y1="48.26" x2="12.7" y2="48.26" width="0.1524" layer="91"/>
+<wire x1="12.7" y1="48.26" x2="12.7" y2="17.78" width="0.1524" layer="91"/>
+<wire x1="12.7" y1="17.78" x2="30.48" y2="17.78" width="0.1524" layer="91"/>
+<pinref part="OCTAVE_SELECT" gate="G$1" pin="A"/>
+<wire x1="22.86" y1="48.26" x2="55.88" y2="48.26" width="0.1524" layer="91"/>
+<wire x1="55.88" y1="48.26" x2="55.88" y2="60.96" width="0.1524" layer="91"/>
+<pinref part="FILTER_CUTOFF" gate="G$1" pin="S"/>
+<wire x1="22.86" y1="48.26" x2="22.86" y2="55.88" width="0.1524" layer="91"/>
+<wire x1="22.86" y1="48.26" x2="22.86" y2="25.4" width="0.1524" layer="91"/>
+<junction x="22.86" y="48.26"/>
+<wire x1="76.2" y1="25.4" x2="30.48" y2="25.4" width="0.1524" layer="91"/>
+<pinref part="JP1" gate="A" pin="7"/>
+<label x="66.04" y="25.4" size="1.778" layer="95"/>
+<wire x1="30.48" y1="25.4" x2="22.86" y2="25.4" width="0.1524" layer="91"/>
+<wire x1="30.48" y1="17.78" x2="30.48" y2="25.4" width="0.1524" layer="91"/>
 </segment>
 </net>
@@
 packages will not be understood (or retained) with this version.
 </note>
+<note version="8.4" severity="warning">
+Since Version 8.4, EAGLE supports properties for SPICE simulation.
+Probes in schematics and SPICE mapping objects found in parts and library devices
+will not be understood with this version. Update EAGLE to the latest version
+for full support of SPICE simulation.
+</note>
 </compatibility>
